File: PCB/wheelBluetooth/wheelBluetooth.kicad_pcb (KiCad board)
At the start: 2 copper layers, 32 parts, among them J1 USB_C_Receptacle_USB2.0, J2 Conn_01x02_Male, J3 Conn_01x06_Male, Q1 A03401A, SW1 SW_Push, SW2 SW_Push, SW3 SW_Push, SW4 SW_Push, SW5 SW_Push, SW6 SW_Push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

Commit message: Schematic update and PCB
Parts:
- added J4: Conn_01x07_Male, Connector_PinSocket_2.54mm:PinSocket_1x07_P2.54mm_Vertical, F.Cu at (185.6, 94.2)
- added J5: Conn_01x07_Male, Connector_PinSocket_2.54mm:PinSocket_1x07_P2.54mm_Vertical, F.Cu at (211.6, 91.9)
- added Q2: MBT3904DW1, Package_TO_SOT_SMD:SOT-363_SC-70-6, F.Cu at (178.8, 70.8)
- added R8: 10K, Resistor_SMD:R_0603_1608Metric, F.Cu at (179.0, 68.4)
- added R9: 10K, Resistor_SMD:R_0603_1608Metric, F.Cu at (178.7, 73.1)
- SW7: footprint josh-buttons-switches:Switch_SMT_SKPMAPE010 -> josh-buttons-switches:SW_Push_KMR2
- moved Q1 67.4 mm to (170.1, 62.2), turned to 90 degrees
- moved D2 67.1 mm to (168.9, 65.5), turned to 180 degrees
- moved C7 62.7 mm to (170.2, 59.4), turned to 180 degrees
- moved C1 58.1 mm to (163.9, 68.2), turned to -90 degrees
- moved C4 58.0 mm to (173.5, 63.2), turned to 180 degrees
- moved F1 57.5 mm to (166.5, 67.7)
- moved U2 55.3 mm to (173.1, 66.4), turned to -90 degrees
- moved SW3 55.1 mm to (215.7, 77.7)
- moved D1 53.1 mm to (169.8, 67.8), turned to 180 degrees
- moved R4 51.5 mm to (172.9, 69.4), turned to 180 degrees
- moved SW6 51.3 mm to (225.9, 85.6)
- moved R2 50.0 mm to (158.5, 67.5), turned to 180 degrees
- moved SW4 47.0 mm to (215.7, 85.6)
- moved SW2 47.0 mm to (205.5, 85.6)
- moved SW5 46.9 mm to (225.9, 77.7)
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Connections:
- U1 pad 10: unconnected-(U1-Pad10) -> /KEY2_1
- U1 pad 11: unconnected-(U1-Pad11) -> /KEY3_1
- U1 pad 12: unconnected-(U1-Pad12) -> /KEY4_1
- U1 pad 13: unconnected-(U1-Pad13) -> /KEY5_1
- U1 pad 14: unconnected-(U1-Pad14) -> /KEY6_1
- U1 pad 25: unconnected-(U1-Pad25) -> /GPIO0
- U1 pad 9: unconnected-(U1-Pad9) -> /KEY1_1
Routing:
- net GND: track 0.00 -> 79.3 mm, vias 0 -> 26
- net +3V3: track 0.00 -> 76.4 mm
- net /VBAT: track 0.00 -> 57.1 mm
- net Net-(R12-Pad2): track 0.00 -> 49.4 mm
- net /nRESET: track 0.00 -> 42.5 mm, vias 0 -> 2
- net +BATT: track 0.00 -> 38.8 mm
- net /DTR: track 0.00 -> 25.7 mm
- net /KEY5: track 0.00 -> 18.6 mm
- net /KEY6_1: track 0.00 -> 18.0 mm
- net /KEY5_1: track 0.00 -> 17.5 mm
- net /KEY4_1: track 0.00 -> 17.1 mm
- net +5V: track 0.00 -> 17.0 mm
- net /KEY1_1: track 0.00 -> 17.0 mm
- net /KEY2_1: track 0.00 -> 16.4 mm
- net /KEY3_1: track 0.00 -> 16.4 mm
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- added copper zone on B.Cu, net GND
- added copper zone on F.Cu, net GND

Commit message: Updated PCB
Parts:
- moved SW7 1.65 mm to (183.7, 73.3), turned to 90 degrees
- moved J1 1.05 mm to (160.3, 61.0)
- moved R12 1.01 mm to (164.9, 95.1)
- moved R4 1.01 mm to (171.9, 69.2)
- moved R6 1.01 mm to (175.3, 67.1)
- moved J2 1.01 mm to (181.3, 62.8)
- moved Q1 1.01 mm to (169.1, 62.1)
- moved C13 1.01 mm to (163.2, 95.1)
- moved D2 1.01 mm to (167.9, 65.3)
- moved U2 1.01 mm to (172.1, 66.2)
- moved C1 1.01 mm to (163.0, 68.0)
- moved C10 1.01 mm to (175.1, 60.6)
- moved C4 1.01 mm to (172.5, 63.1)
- moved C7 1.01 mm to (169.2, 59.2)
- moved D1 1.01 mm to (168.8, 67.6)
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Routing:
- net /VBAT: track 57.1 -> 59.4 mm
- net GND: track 79.3 -> 80.8 mm
- net Net-(R12-Pad2): track 49.4 -> 48.4 mm
- removed copper zone on F.Cu, net GND
Other:
- board outline added: 81.5 x 40.5 mm

Commit message: PCB graphics
Parts:
- added G***: LOGO, LOGO, B.Cu at (216.2, 81.7)
- added G***: LOGO, LOGO, B.Cu at (242.7, 69.8)
- added G***: LOGO, LOGO, B.Cu at (170.0, 77.8)
- added G***: LOGO, LOGO, B.Cu at (217.2, 75.2)
- added G***: LOGO, LOGO, B.Cu at (253.0, 70.1)
- moved SW1 5.16 mm to (200.5, 76.6)
- moved SW2 4.18 mm to (201.5, 84.6)
- moved SW3 3.39 mm to (212.5, 76.6)
- moved SW4 2.43 mm to (213.5, 84.6)
- moved J5 2.38 mm to (209.6, 90.6)
- moved SW5 1.76 mm to (224.5, 76.6)
- moved SW6 1.07 mm to (225.5, 84.6)
- moved R8 0.31 mm to (177.7, 68.3)
- moved U3 0.23 mm to (172.5, 60.5)
- moved C10 0.22 mm to (175.3, 60.7)
- moved R5 0.22 mm to (175.1, 64.1)
- moved R6 0.20 mm to (175.1, 67.2)
- moved C7 0.19 mm to (169.1, 59.3)
- moved C4 0.18 mm to (172.5, 63.2)
- moved C3 0.18 mm to (160.9, 96.1)
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Routing:
- net /nRESET: track 42.5 -> 32.8 mm
- net GND: track 80.8 -> 72.7 mm
- net /KEY5: track 18.6 -> 20.8 mm
- net /KEY6: track 10.2 -> 11.6 mm
- net /KEY3: track 16.3 -> 15.6 mm
- net /KEY4_1: track 17.1 -> 17.8 mm
- net /KEY5_1: track 17.5 -> 18.2 mm
- net /KEY6_1: track 18.0 -> 18.6 mm
- net /KEY3_1: track 16.4 -> 17.0 mm
- net /DTR: track 25.7 -> 26.3 mm
- net /KEY2: track 7.41 -> 7.94 mm
Other:
- board size 81.5 x 40.5 mm -> 82.8 x 40.5 mm
- board text added: "M'"
- board text added: "Ranger"
- board text added: "bing"
- board text added: "opsbinxu"

Commit message: Update PCB
Parts:
- removed the G*** at (170.0, 77.8)
- added G***: LOGO, LOGO, B.Cu at (170.0, 64.6)
- added G***: LOGO, LOGO, B.Cu at (173.1, 85.3)
- moved G*** 41.8 mm to (223.3, 40.6)
- moved G*** 41.8 mm to (213.1, 40.3)
- moved J5 0.32 mm to (209.3, 90.5)
Other:
- board text added: "M'Ranger"
- board text removed: "M'"
- board text removed: "Ranger"

Commit message: Update PCB
Parts:
- removed the G*** at (213.1, 40.3)
- removed the G*** at (223.3, 40.6)
- moved SW5 31.5 mm to (194.0, 68.9), turned to 90 degrees
- moved SW6 28.8 mm to (202.0, 67.9), turned to 90 degrees
- moved G*** 26.8 mm to (170.3, 91.4), turned to 0 degrees
- moved G*** 23.3 mm to (193.9, 76.0), turned to -90 degrees
- moved SW3 19.0 mm to (194.0, 80.9), turned to 90 degrees
- moved SW1 17.5 mm to (194.0, 92.9), turned to 90 degrees
- moved G*** 16.6 mm to (200.4, 76.9), turned to -90 degrees
- moved G*** 14.9 mm to (166.2, 72.1), turned to 0 degrees
- moved SW4 12.4 mm to (202.0, 79.9), turned to 90 degrees
- moved SW2 7.32 mm to (202.0, 91.9), turned to 90 degrees
- moved J5 4.50 mm to (208.1, 86.2), turned to 180 degrees
- moved SW7 1.30 mm to (183.7, 72.0), turned to -90 degrees
- moved F1 0.59 mm to (165.5, 68.1)
- moved R3 0.46 mm to (168.8, 69.6)
- moved U3 0.44 mm to (172.6, 60.9)
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Routing:
- net GND: track 73.0 -> 50.2 mm, vias 26 -> 28
- net /VBAT: track 59.6 -> 37.7 mm
- net +3V3: track 76.4 -> 90.0 mm
- net /KEY3_1: track 17.0 -> 27.4 mm
- net /KEY6: track 11.9 -> 15.5 mm
- net /KEY5: track 21.1 -> 24.2 mm
- net Net-(R12-Pad2): track 48.4 -> 45.5 mm, vias 0 -> 2
- net /KEY4: track 7.21 -> 9.47 mm
- net /KEY3: track 15.9 -> 17.6 mm
- net /KEY6_1: track 18.6 -> 19.6 mm
- net /KEY5_1: track 18.2 -> 19.1 mm
- net /KEY2: track 7.73 -> 6.98 mm
- net /nRESET: track 32.8 -> 32.1 mm
- net Net-(C1-Pad1): track 11.6 -> 12.2 mm
- net /KEY1: track 15.4 -> 14.8 mm
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Other:
- board size 82.8 x 40.5 mm -> 57.5 x 40.5 mm

Commit message: Fixed reset circuit
Connections:
- R12 pad 2: Net-(R12-Pad2) -> /nRESET
- SW7 pad 2: Net-(R12-Pad2) -> /nRESET
Routing:
- net /nRESET: track 32.1 -> 79.2 mm, vias 2 -> 4
- net Net-(R12-Pad2): track 45.5 -> 0.00 mm, vias 2 -> 0
- net /KEY3_1: track 27.4 -> 0.00 mm
- net /KEY1: track 14.8 -> 42.1 mm
