File: PCB/wheelBluetooth/wheelBluetooth.kicad_sch (KiCad schematic)
At the start: 32 parts, among them J1 USB_C_Receptacle_USB2.0, J2 Conn_01x02_Male, J3 Conn_01x06_Male, Q1 A03401A, SW1 SW_Push, SW2 SW_Push, SW3 SW_Push, SW4 SW_Push, SW5 SW_Push, SW6 SW_Push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

Commit message: Schematic
Parts:
- added J? (x2): Conn_01x07_Male, symbol Connector:Conn_01x07_Male
Connections:
- net GND: now also J?.7 (Pin_7), J?.7 (Pin_7)
- net KEY1: now also J?.1 (Pin_1)
- net KEY2: now also J?.2 (Pin_2)
- net KEY3: now also J?.3 (Pin_3)
- net KEY4: now also J?.4 (Pin_4)
- net KEY5: now also J?.5 (Pin_5)
- net KEY6: now also J?.6 (Pin_6)
- new net KEY1_1: J?.1 (Pin_1)
- new net KEY2_1: J?.2 (Pin_2)
- new net KEY3_1: J?.3 (Pin_3)
- new net KEY4_1: J?.4 (Pin_4)
- new net KEY5_1: J?.5 (Pin_5)
- new net KEY6_1: J?.6 (Pin_6)
Changed lines of the file:
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@@
+    (stroke (width 0) (type solid) (color 0 0 0 0))
+  )
+  (wire (pts (xy 69.85 154.94) (xy 60.96 154.94))
+    (stroke (width 0) (type solid) (color 0 0 0 0))
+  )
+  (wire (pts (xy 69.85 157.48) (xy 60.96 157.48))
+    (stroke (width 0) (type solid) (color 0 0 0 0))
+  )
+  (wire (pts (xy 69.85 160.02) (xy 60.96 160.02))
+    (stroke (width 0) (type solid) (color 0 0 0 0))
+  )
+  (wire (pts (xy 69.85 162.56) (xy 60.96 162.56))
+    (stroke (width 0) (type solid) (color 0 0 0 0))
+  )
+  (wire (pts (xy 69.85 165.1) (xy 60.96 165.1))
+    (stroke (width 0) (type solid) (color 0 0 0 0))
+  )
+  (wire (pts (xy 69.85 167.64) (xy 60.96 167.64))
     (stroke (width 0) (type solid) (color 0 0 0 0))
   )
@@
     (stroke (width 0) (type solid) (color 0 0 0 0))
   )
-  (wire (pts (xy 72.39 161.29) (xy 63.5 161.29))
-    (stroke (width 0) (type solid) (color 0 0 0 0))
-  )
-  (wire (pts (xy 72.39 163.83) (xy 63.5 163.83))
-    (stroke (width 0) (type solid) (color 0 0 0 0))
-  )
-  (wire (pts (xy 72.39 166.37) (xy 63.5 166.37))
-    (stroke (width 0) (type solid) (color 0 0 0 0))
-  )
-  (wire (pts (xy 72.39 168.91) (xy 63.5 168.91))
-    (stroke (width 0) (type solid) (color 0 0 0 0))
-  )
-  (wire (pts (xy 72.39 171.45) (xy 63.5 171.45))
-    (stroke (width 0) (type solid) (color 0 0 0 0))
-  )
-  (wire (pts (xy 72.39 173.99) (xy 63.5 173.99))
-    (stroke (width 0) (type solid) (color 0 0 0 0))
-  )
   (wire (pts (xy 73.66 35.56) (xy 77.47 35.56))
     (stroke (width 0) (type solid) (color 0 0 0 0))
@@
     (stroke (width 0) (type solid) (color 0 0 0 0))
   )
+  (wire (pts (xy 92.075 158.75) (xy 83.185 158.75))
+    (stroke (width 0) (type solid) (color 0 0 0 0))
+  )
+  (wire (pts (xy 92.075 161.29) (xy 83.185 161.29))
+    (stroke (width 0) (type solid) (color 0 0 0 0))
+  )
+  (wire (pts (xy 92.075 163.83) (xy 83.185 163.83))
+    (stroke (width 0) (type solid) (color 0 0 0 0))
+  )
+  (wire (pts (xy 92.075 166.37) (xy 83.185 166.37))
+    (stroke (width 0) (type solid) (color 0 0 0 0))
+  )
+  (wire (pts (xy 92.075 168.91) (xy 83.185 168.91))
+    (stroke (width 0) (type solid) (color 0 0 0 0))
+  )
+  (wire (pts (xy 92.075 171.45) (xy 83.185 171.45))
+    (stroke (width 0) (type solid) (color 0 0 0 0))
+  )
   (wire (pts (xy 119.38 93.98) (xy 127 93.98))
     (stroke (width 0) (type solid) (color 0 0 0 0))
@@
   )
   (wire (pts (xy 167.64 186.69) (xy 167.64 187.96))
+    (stroke (width 0) (type solid) (color 0 0 0 0))
+  )
+  (wire (pts (xy 177.165 121.92) (xy 168.275 121.92))
+    (stroke (width 0) (type solid) (color 0 0 0 0))
+  )
+  (wire (pts (xy 177.165 124.46) (xy 168.275 124.46))
+    (stroke (width 0) (type solid) (color 0 0 0 0))
+  )
+  (wire (pts (xy 177.165 127) (xy 168.275 127))
+    (stroke (width 0) (type solid) (color 0 0 0 0))
+  )
+  (wire (pts (xy 177.165 129.54) (xy 168.275 129.54))
+    (stroke (width 0) (type solid) (color 0 0 0 0))
+  )
+  (wire (pts (xy 177.165 132.08) (xy 168.275 132.08))
+    (stroke (width 0) (type solid) (color 0 0 0 0))
+  )
+  (wire (pts (xy 177.165 134.62) (xy 168.275 134.62))
     (stroke (width 0) (type solid) (color 0 0 0 0))
   )
@@
     (effects (font (size 1.27 1.27)) (justify right bottom))
   )
-  (label "KEY1" (at 72.39 161.29 180)
-    (effects (font (size 1.27 1.27)) (justify right bottom))
-  )
-  (label "KEY2" (at 72.39 163.83 180)
-    (effects (font (size 1.27 1.27)) (justify right bottom))
-  )
-  (label "KEY3" (at 72.39 166.37 180)
-    (effects (font (size 1.27 1.27)) (justify right bottom))
-  )
-  (label "KEY4" (at 72.39 168.91 180)
-    (effects (font (size 1.27 1.27)) (justify right bottom))
-  )
-  (label "KEY5" (at 72.39 171.45 180)
-    (effects (font (size 1.27 1.27)) (justify right bottom))
-  )
-  (label "KEY6" (at 72.39 173.99 180)
+  (label "KEY1_1" (at 69.85 154.94 180)
+    (effects (font (size 1.27 1.27)) (justify right bottom))
+  )
+  (label "KEY2_1" (at 69.85 157.48 180)
+    (effects (font (size 1.27 1.27)) (justify right bottom))
+  )
+  (label "KEY3_1" (at 69.85 160.02 180)
+    (effects (font (size 1.27 1.27)) (justify right bottom))
+  )
+  (label "KEY4_1" (at 69.85 162.56 180)
+    (effects (font (size 1.27 1.27)) (justify right bottom))
+  )
+  (label "KEY5_1" (at 69.85 165.1 180)
+    (effects (font (size 1.27 1.27)) (justify right bottom))
+  )
+  (label "KEY6_1" (at 69.85 167.64 180)
+    (effects (font (size 1.27 1.27)) (justify right bottom))
+  )
+  (label "KEY1_1" (at 92.075 158.75 180)
+    (effects (font (size 1.27 1.27)) (justify right bottom))
+  )
+  (label "KEY2_1" (at 92.075 161.29 180)
+    (effects (font (size 1.27 1.27)) (justify right bottom))
+  )
+  (label "KEY3_1" (at 92.075 163.83 180)
+    (effects (font (size 1.27 1.27)) (justify right bottom))
+  )
+  (label "KEY4_1" (at 92.075 166.37 180)
+    (effects (font (size 1.27 1.27)) (justify right bottom))
+  )
+  (label "KEY5_1" (at 92.075 168.91 180)
+    (effects (font (size 1.27 1.27)) (justify right bottom))
+  )
+  (label "KEY6_1" (at 92.075 171.45 180)
     (effects (font (size 1.27 1.27)) (justify right bottom))
   )
@@
     (effects (font (size 1.27 1.27)) (justify right bottom))
   )
+  (label "KEY1" (at 177.165 121.92 180)
+    (effects (font (size 1.27 1.27)) (justify right bottom))
+  )
+  (label "KEY2" (at 177.165 124.46 180)
+    (effects (font (size 1.27 1.27)) (justify right bottom))
+  )
+  (label "KEY3" (at 177.165 127 180)
+    (effects (font (size 1.27 1.27)) (justify right bottom))
+  )
+  (label "KEY4" (at 177.165 129.54 180)
+    (effects (font (size 1.27 1.27)) (justify right bottom))
+  )
+  (label "KEY5" (at 177.165 132.08 180)
+    (effects (font (size 1.27 1.27)) (justify right bottom))
+  )
+  (label "KEY6" (at 177.165 134.62 180)
+    (effects (font (size 1.27 1.27)) (justify right bottom))
+  )
   (label "KEY1" (at 193.04 125.73 270)
     (effects (font (size 1.27 1.27)) (justify right bottom))
@@
     (pin "1")
   )
+  (symbol (lib_id "power:GND") (at 83.185 173.99 90) (mirror x) (unit 1)
+    (in_bom yes) (on_board yes)
+    (property "Reference" "#PWR?" (id 0) (at 89.535 173.99 0)
+      (effects (font (size 1.27 1.27)) hide)
+    )
+    (property "Value" "GND" (id 1) (at 89.7889 173.511 90)
+      (effects (font (size 1.27 1.27)) (justify left))
+    )
+    (property "Footprint" "" (id 2) (at 83.185 173.99 0)
+      (effects (font (size 1.27 1.27)) hide)
+    )
+    (property "Datasheet" "" (id 3) (at 83.185 173.99 0)
+      (effects (font (size 1.27 1.27)) hide)
+    )
+    (pin "1")
+  )
   (symbol (lib_id "power:GND") (at 102.87 156.21 0) (unit 1)
     (in_bom yes) (on_board yes) (fields_autoplaced)
@@
     )
     (property "Datasheet" "" (id 3) (at 167.64 187.96 0)
+      (effects (font (size 1.27 1.27)) hide)
+    )
+    (pin "1")
+  )
+  (symbol (lib_id "power:GND") (at 168.275 137.16 90) (mirror x) (unit 1)
+    (in_bom yes) (on_board yes)
+    (property "Reference" "#PWR?" (id 0) (at 174.625 137.16 0)
+      (effects (font (size 1.27 1.27)) hide)
+    )
+    (property "Value" "GND" (id 1) (at 174.8789 136.681 90)
+      (effects (font (size 1.27 1.27)) (justify left))
+    )
+    (property "Footprint" "" (id 2) (at 168.275 137.16 0)
+      (effects (font (size 1.27 1.27)) hide)
+    )
+    (property "Datasheet" "" (id 3) (at 168.275 137.16 0)
       (effects (font (size 1.27 1.27)) hide)
     )
@@
     (pin "5")
     (pin "6")
+  )
+  (symbol (lib_id "Connector:Conn_01x07_Male") (at 78.105 166.37 0) (unit 1)
+    (in_bom yes) (on_board yes)
+    (property "Reference" "J?" (id 0) (at 80.7974 152.6244 0))
+    (property "Value" "Conn_01x07_Male" (id 1) (at 80.7974 155.3995 0))
+    (property "Footprint" "" (id 2) (at 78.105 166.37 0)
+      (effects (font (size 1.27 1.27)) hide)
+    )
+    (property "Datasheet" "~" (id 3) (at 78.105 166.37 0)
+      (effects (font (size 1.27 1.27)) hide)
+    )
+    (pin "1")
+    (pin "2")
+    (pin "3")
+    (pin "4")
+    (pin "5")
+    (pin "6")
+    (pin "7")
+  )
+  (symbol (lib_id "Connector:Conn_01x07_Male") (at 163.195 129.54 0) (unit 1)
+    (in_bom yes) (on_board yes)
+    (property "Reference" "J?" (id 0) (at 165.8874 115.7944 0))
+    (property "Value" "Conn_01x07_Male" (id 1) (at 165.8874 118.5695 0))
+    (property "Footprint" "" (id 2) (at 163.195 129.54 0)
+      (effects (font (size 1.27 1.27)) hide)
+    )
+    (property "Datasheet" "~" (id 3) (at 163.195 129.54 0)
+      (effects (font (size 1.27 1.27)) hide)
+    )
+    (pin "1")
+    (pin "2")
+    (pin "3")
+    (pin "4")
+    (pin "5")
+    (pin "6")
+    (pin "7")
   )
   (symbol (lib_id "Transistor_FET:TP0610T") (at 224.79 33.02 0) (unit 1)
@@
       (reference "#PWR0119") (unit 1) (value "GND") (footprint "")
     )
+    (path "/40733706-8777-40b7-9aaa-ef42212bd818"
+      (reference "#PWR?") (unit 1) (value "GND") (footprint "")
+    )
+    (path "/b4ab01c9-edc5-4e25-813a-b4767e8b1ad8"
+      (reference "#PWR?") (unit 1) (value "GND") (footprint "")
+    )
     (path "/20bb962e-b864-402d-b62e-20bdd7b90164"
       (reference "C1") (unit 1) (value "10u") (footprint "Capacitor_SMD:C_0603_1608Metric")
@@
       (reference "J3") (unit 1) (value "Conn_01x06_Male") (footprint "josh-connectors:6_PIN_THT_Staggered")
     )
+    (path "/5ed64efc-21f1-4088-8abd-5fed7435f272"
+      (reference "J?") (unit 1) (value "Conn_01x07_Male") (footprint "")
+    )
+    (path "/635b1f5b-beab-4dba-a362-8a3b90266f0c"
+      (reference "J?") (unit 1) (value "Conn_01x07_Male") (footprint "")
+    )
     (path "/48f23001-4d0a-4ff0-817e-d51407ce7123"

Commit message: Schematic update and PCB
Parts:
- added Q2: MBT3904DW1, Package_TO_SOT_SMD:SOT-363_SC-70-6, symbol Transistor_BJT:FFB2222A
- added R8, R9: 10K, Resistor_SMD:R_0603_1608Metric, symbol Device:R
- J4, J5: renamed from J?; footprint (none) -> Connector_PinSocket_2.54mm:PinSocket_1x07_P2.54mm_Vertical
- SW7: footprint josh-buttons-switches:Switch_SMT_SKPMAPE010 -> josh-buttons-switches:SW_Push_KMR2
Connections:
- net DTR: now also Q2.1 (E1), R9.1
- net KEY1_1: now also U1.9 (IO33)
- net KEY2_1: now also U1.10 (IO25)
- net KEY3_1: now also U1.11 (IO26)
- net KEY4_1: now also U1.12 (IO27)
- net KEY5_1: now also U1.13 (IO14)
- net KEY6_1: now also U1.14 (IO12)
- net RTS: now also Q2.4 (E2), R8.1
- net nRESET: now also Q2.3 (C2)
- net GPIO0: now reaches U1.25 (IO0)
- net GPIO0: now also Q2.6 (C1)
- new net: Q2.5 (B2), R9.2
- new net: Q2.2 (B1), R8.2
- no-connect marks 16 -> 15
Other:
- note added: "CPU side"
- note added: "Switch side"
- moved on the sheet: C13, J2, J3, J4, J5, R12, SW7

Commit message: Fixed reset circuit
Connections:
- net nRESET: now also R12.2, SW7.2
Other:
- moved on the sheet: C13, SW7
Changed lines of the file:
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@@
   (junction (at 75.565 137.795) (diameter 1.016) (color 0 0 0 0))
   (junction (at 77.47 35.56) (diameter 1.016) (color 0 0 0 0))
+  (junction (at 140.335 94.615) (diameter 1.016) (color 0 0 0 0))
   (junction (at 147.955 94.615) (diameter 1.016) (color 0 0 0 0))
   (junction (at 157.48 38.1) (diameter 1.016) (color 0 0 0 0))
@@
     (stroke (width 0) (type solid) (color 0 0 0 0))
   )
+  (wire (pts (xy 140.335 94.615) (xy 140.335 93.345))
+    (stroke (width 0) (type solid) (color 0 0 0 0))
+  )
   (wire (pts (xy 140.335 94.615) (xy 147.955 94.615))
     (stroke (width 0) (type solid) (color 0 0 0 0))
   )
+  (wire (pts (xy 140.335 96.52) (xy 140.335 94.615))
+    (stroke (width 0) (type solid) (color 0 0 0 0))
+  )
   (wire (pts (xy 143.51 27.94) (xy 143.51 33.02))
     (stroke (width 0) (type solid) (color 0 0 0 0))
@@
     (stroke (width 0) (type solid) (color 0 0 0 0))
   )
-  (wire (pts (xy 147.955 94.615) (xy 147.955 95.885))
+  (wire (pts (xy 147.955 94.615) (xy 147.955 99.06))
     (stroke (width 0) (type solid) (color 0 0 0 0))
   )
@@
     (pin "1")
   )
-  (symbol (lib_id "power:GND") (at 140.335 103.505 0) (unit 1)
-    (in_bom yes) (on_board yes) (fields_autoplaced)
-    (property "Reference" "#PWR038" (id 0) (at 140.335 109.855 0)
-      (effects (font (size 1.27 1.27)) hide)
-    )
-    (property "Value" "GND" (id 1) (at 140.335 108.0676 0))
-    (property "Footprint" "" (id 2) (at 140.335 103.505 0)
-      (effects (font (size 1.27 1.27)) hide)
-    )
-    (property "Datasheet" "" (id 3) (at 140.335 103.505 0)
+  (symbol (lib_id "power:GND") (at 140.335 106.68 0) (unit 1)
+    (in_bom yes) (on_board yes) (fields_autoplaced)
+    (property "Reference" "#PWR038" (id 0) (at 140.335 113.03 0)
+      (effects (font (size 1.27 1.27)) hide)
+    )
+    (property "Value" "GND" (id 1) (at 140.335 111.2426 0))
+    (property "Footprint" "" (id 2) (at 140.335 106.68 0)
+      (effects (font (size 1.27 1.27)) hide)
+    )
+    (property "Datasheet" "" (id 3) (at 140.335 106.68 0)
       (effects (font (size 1.27 1.27)) hide)
     )
@@
     (pin "1")
   )
-  (symbol (lib_id "power:GND") (at 147.955 103.505 0) (unit 1)
-    (in_bom yes) (on_board yes) (fields_autoplaced)
-    (property "Reference" "#PWR039" (id 0) (at 147.955 109.855 0)
-      (effects (font (size 1.27 1.27)) hide)
-    )
-    (property "Value" "GND" (id 1) (at 147.955 108.0676 0))
-    (property "Footprint" "" (id 2) (at 147.955 103.505 0)
-      (effects (font (size 1.27 1.27)) hide)
-    )
-    (property "Datasheet" "" (id 3) (at 147.955 103.505 0)
+  (symbol (lib_id "power:GND") (at 147.955 106.68 0) (unit 1)
+    (in_bom yes) (on_board yes) (fields_autoplaced)
+    (property "Reference" "#PWR039" (id 0) (at 147.955 113.03 0)
+      (effects (font (size 1.27 1.27)) hide)
+    )
+    (property "Value" "GND" (id 1) (at 147.955 111.2426 0))
+    (property "Footprint" "" (id 2) (at 147.955 106.68 0)
+      (effects (font (size 1.27 1.27)) hide)
+    )
+    (property "Datasheet" "" (id 3) (at 147.955 106.68 0)
       (effects (font (size 1.27 1.27)) hide)
     )
@@
     (pin "2")
   )
-  (symbol (lib_id "Device:C") (at 147.955 99.695 0) (unit 1)
-    (in_bom yes) (on_board yes)
-    (property "Reference" "C13" (id 0) (at 150.8761 98.7865 0)
-      (effects (font (size 1.27 1.27)) (justify left))
-    )
-    (property "Value" "1u" (id 1) (at 150.8761 101.5616 0)
-      (effects (font (size 1.27 1.27)) (justify left))
-    )
-    (property "Footprint" "Capacitor_SMD:C_0603_1608Metric" (id 2) (at 148.9202 103.505 0)
-      (effects (font (size 1.27 1.27)) hide)
-    )
-    (property "Datasheet" "~" (id 3) (at 147.955 99.695 0)
+  (symbol (lib_id "Device:C") (at 147.955 102.87 0) (unit 1)
+    (in_bom yes) (on_board yes)
+    (property "Reference" "C13" (id 0) (at 150.8761 101.9615 0)
+      (effects (font (size 1.27 1.27)) (justify left))
+    )
+    (property "Value" "1u" (id 1) (at 150.8761 104.7366 0)
+      (effects (font (size 1.27 1.27)) (justify left))
+    )
+    (property "Footprint" "Capacitor_SMD:C_0603_1608Metric" (id 2) (at 148.9202 106.68 0)
+      (effects (font (size 1.27 1.27)) hide)
+    )
+    (property "Datasheet" "~" (id 3) (at 147.955 102.87 0)
       (effects (font (size 1.27 1.27)) hide)
     )
@@
     (pin "2")
   )
-  (symbol (lib_id "Switch:SW_Push") (at 140.335 98.425 90) (unit 1)
-    (in_bom yes) (on_board yes)
-    (property "Reference" "SW7" (id 0) (at 128.7781 97.5165 90)
+  (symbol (lib_id "Switch:SW_Push") (at 140.335 101.6 90) (unit 1)
+    (in_bom yes) (on_board yes)
+    (property "Reference" "SW7" (id 0) (at 128.7781 100.6915 90)
       (effects (font (size 1.27 1.27)) (justify right))
     )
-    (property "Value" "SW_Push" (id 1) (at 128.7781 100.2916 90)
+    (property "Value" "SW_Push" (id 1) (at 128.7781 103.4666 90)
       (effects (font (size 1.27 1.27)) (justify right))
     )
-    (property "Footprint" "josh-buttons-switches:SW_Push_KMR2" (id 2) (at 135.255 98.425 0)
-      (effects (font (size 1.27 1.27)) hide)
-    )
-    (property "Datasheet" "~" (id 3) (at 135.255 98.425 0)
-      (effects (font (size 1.27 1.27)) hide)
-    )
+    (property "Footprint" "josh-buttons-switches:SW_Push_KMR2" (id 2) (at 135.255 101.6 0)
+      (effects (font (size 1.27 1.27)) hide)
+    )
+    (property "Datasheet" "~" (id 3) (at 135.255 101.6 0)
+      (effects (font (size 1.27 1.27)) hide)
+    )
